File: board/StairLights_screw.brd (EAGLE design)
At the start: 83.7 x 51.9 mm, 27 parts, among them J1 1,2, J2 3,4, J3 5,6, J4 7, 12V, J5 SIGN_TOP, J7 SIGN_BOTTOM, J8 SIGN_PWR, M1 ARDUINO-PRO-MINI-5.0VNOSIDEPI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

Commit message: Исправлена ошибка с номиналом потенциометра
Parts:
- R11: value 10k -> 100k
Changed lines of the file:
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@@
 <attribute name="VALUE" x="7.493" y="19.6916" size="0.6096" layer="27" font="vector" ratio="20" rot="R270" align="top-center"/>
 </element>
-<element name="R11" library="pot" library_urn="urn:adsk.eagle:library:331" package="S64W" package3d_urn="urn:adsk.eagle:package:22708/1" value="10k" x="32.766" y="31.75" smashed="yes" rot="R90">
+<element name="R11" library="pot" library_urn="urn:adsk.eagle:library:331" package="S64W" package3d_urn="urn:adsk.eagle:package:22708/1" value="100k" x="32.766" y="31.75" smashed="yes" rot="R90">
 <attribute name="NAME" x="28.6258" y="26.924" size="1.27" layer="25" ratio="10" rot="R90"/>
 <attribute name="VALUE" x="35.687" y="26.9494" size="1.27" layer="27" ratio="10" rot="R90"/>
